Commit message: Multiple tiny fixes: script now runs!

File: assets/robots/so101.urdf (robot description, URDF)
Before this commit: robot so100, 9 links, 8 joints
Joints:
- removed joint 1
- removed joint 2
- removed joint 3
- removed joint 4
- removed joint 5
- removed joint 6
- added joint elbow_flex: type revolute, parent upper_arm, child lower_arm, origin xyz=-0.11257 -0.028 2.09886e-16 rpy=-3.63608e-16 8.74301e-16 1.5708, axis 0 0 1, limit lower=-1.74533 upper=1.5708 effort=10 velocity=10
- added joint gripper: type revolute, parent gripper, child moving_jaw_so101_v1, origin xyz=0.0202 0.0188 -0.0234 rpy=1.5708 -5.24284e-08 -1.41553e-15, axis 0 0 1, limit lower=-0.174533 upper=1.74533 effort=10 velocity=10
- added joint shoulder_lift: type revolute, parent shoulder, child upper_arm, origin xyz=-0.0303992 -0.0182778 -0.0542 rpy=-1.5708 -1.5708 0, axis 0 0 1, limit lower=-1.74533 upper=1.74533 effort=10 velocity=10
- added joint shoulder_pan: type revolute, parent base, child shoulder, origin xyz=-0.124202 -0.168068 0.0948817 rpy=3.14159 4.18253e-17 -3.14159, axis 0 0 1, limit lower=-1.91986 upper=1.91986 effort=10 velocity=10
- added joint wrist_flex: type revolute, parent lower_arm, child wrist, origin xyz=-0.1349 0.0052 8.44651e-17 rpy=4.02456e-15 8.67362e-16 -1.5708, axis 0 0 1, limit lower=-1.65806 upper=1.65806 effort=10 velocity=10
- added joint wrist_roll: type revolute, parent wrist, child gripper, origin xyz=2.77556e-16 -0.0611 0.0181 rpy=1.5708 0.0486795 3.14159, axis 0 0 1, limit lower=-2.74385 upper=2.84121 effort=10 velocity=10

Commit message: New urdf file

File: assets/robots/so101.urdf (robot description, URDF)
Before this commit: robot so100, 9 links, 8 joints
Links:
- removed link base
- removed link baseframe
- removed link gripper
- removed link gripperframe
- removed link lower_arm
- removed link moving_jaw_so101_v1
- removed link shoulder
- removed link upper_arm
- removed link wrist
- added link base_link, mass 0.147; collision mesh filename=assets/base_motor_holder_so101_v1.stl; collision mesh filename=assets/base_so101_v2.stl
- added link gripper_frame_link, mass 1e-9
- added link gripper_link, mass 0.087; collision mesh filename=assets/sts3215_03a_v1.stl; collision mesh filename=assets/wrist_roll_follower_so101_v1.stl
- added link lower_arm_link, mass 0.104; collision mesh filename=assets/motor_holder_so101_wrist_v1.stl; collision mesh filename=assets/sts3215_03a_v1.stl
- added link moving_jaw_so101_v1_link, mass 0.012; collision mesh filename=assets/moving_jaw_so101_v1.stl; visual mesh filename=assets/moving_jaw_so101_v1.stl
- added link shoulder_link, mass 0.100006; collision mesh filename=assets/motor_holder_so101_base_v1.stl; collision mesh filename=assets/rotation_pitch_so101_v1.stl
- added link upper_arm_link, mass 0.103; collision mesh filename=assets/sts3215_03a_v1.stl; collision mesh filename=assets/upper_arm_so101_v1.stl
- added link wrist_link, mass 0.079; collision mesh filename=assets/sts3215_03a_no_horn_v1.stl; collision mesh filename=assets/wrist_roll_pitch_so101_v2.stl
Joints:
- removed joint baseframe_frame
- removed joint gripperframe_frame
- added joint gripper_frame_joint: type fixed, parent gripper_link, child gripper_frame_link, origin xyz=-0.0079 -0.000218121 -0.0981274 rpy=0 3.14159 0, axis 0 0 0
- joint elbow_flex: child lower_arm -> lower_arm_link; limit lower=-1.74533 upper=1.5708 effort=10 velocity=10 -> lower=-1.69 upper=1.69 effort=10 velocity=10; origin xyz=-0.11257 -0.028 2.09886e-16 rpy=-3.63608e-16 8.74301e-16 1.5708 -> xyz=-0.11257 -0.028 1.73763e-16 rpy=-3.63608e-16 8.74301e-16 1.5708; parent upper_arm -> upper_arm_link
- joint gripper: child moving_jaw_so101_v1 -> moving_jaw_so101_v1_link; parent gripper -> gripper_link
- joint shoulder_lift: child upper_arm -> upper_arm_link; parent shoulder -> shoulder_link
- joint shoulder_pan: child shoulder -> shoulder_link; origin xyz=-0.124202 -0.168068 0.0948817 rpy=3.14159 4.18253e-17 -3.14159 -> xyz=0.0388353 -8.97657e-09 0.0624 rpy=3.14159 4.18253e-17 -3.14159; parent base -> base_link
- joint wrist_flex: child wrist -> wrist_link; origin xyz=-0.1349 0.0052 8.44651e-17 rpy=4.02456e-15 8.67362e-16 -1.5708 -> xyz=-0.1349 0.0052 3.62355e-17 rpy=4.02456e-15 8.67362e-16 -1.5708; parent lower_arm -> lower_arm_link
- joint wrist_roll: child gripper -> gripper_link; origin xyz=2.77556e-16 -0.0611 0.0181 rpy=1.5708 0.0486795 3.14159 -> xyz=5.55112e-17 -0.0611 0.0181 rpy=1.5708 0.0486795 3.14159; parent wrist -> wrist_link
